Commit message: Update rover_arm.xacro

File: rover_arm_pkg/urdf/rover_arm.xacro (robot description, xacro)
@@ -0,0 +1,114 @@
+<?xml version="1.0"?>
+<robot xmlns:xacro="http://www.ros.org/wiki/xacro" name="rover_arm">
+  <xacro:property name="base_height" value="0.05" />
+  <xacro:property name="link1_len"   value="0.10" /> <xacro:property name="link2_len"   value="0.20" /> <xacro:property name="link3_len"   value="0.15" /> <xacro:property name="link4_len"   value="0.05" /> <xacro:property name="gripper_len" value="0.08" /> <xacro:property name="link_radius" value="0.02" /> <material name="grey">
+    <color rgba="0.5 0.5 0.5 1.0"/>
+  </material>
+  <material name="orange">
+    <color rgba="1.0 0.4 0.0 1.0"/>
+  </material>
+  <link name="base_link">
+    <visual>
+      <geometry>
+        <box size="0.1 0.1 ${base_height}"/>
+      </geometry>
+      <origin xyz="0 0 ${base_height/2}" rpy="0 0 0"/>
+      <material name="grey"/>
+    </visual>
+    <collision>
+      <geometry>
+        <box size="0.1 0.1 ${base_height}"/>
+      </geometry>
+    </collision>
+  </link>
+  <link name="link1">
+    <visual>
+      <geometry>
+        <cylinder radius="${link_radius}" length="${link1_len}"/>
+      </geometry>
+      <origin xyz="0 0 ${link1_len/2}" rpy="0 0 0"/>
+      <material name="orange"/>
+    </visual>
+  </link>
+  <joint name="joint1" type="revolute">
+    <parent link="base_link"/>
+    <child link="link1"/>
+    <origin xyz="0 0 ${base_height}" rpy="0 0 0"/>
+    <axis xyz="0 0 1"/>
+    <limit lower="-3.14" upper="3.14" effort="2.0" velocity="1.0"/>
+  </joint>
+  <link name="link2">
+    <visual>
+      <geometry>
+        <cylinder radius="${link_radius}" length="${link2_len}"/>
+      </geometry>
+      <origin xyz="0 0 ${link2_len/2}" rpy="0 1.5708 0"/> <material name="grey"/>
+    </visual>
+  </link>
+  <joint name="joint2" type="revolute">
+    <parent link="link1"/>
+    <child link="link2"/>
+    <origin xyz="0 0 ${link1_len}" rpy="0 0 0"/>
+    <axis xyz="0 1 0"/> <limit lower="-1.57" upper="1.57" effort="2.0" velocity="1.0"/>
+  </joint>
+  <link name="link3">
+    <visual>
+      <geometry>
+        <cylinder radius="${link_radius}" length="${link3_len}"/>
+      </geometry>
+      <origin xyz="0 0 ${link3_len/2}" rpy="0 1.5708 0"/>
+      <material name="orange"/>
+    </visual>
+  </link>
+  <joint name="joint3" type="revolute">
+    <parent link="link2"/>
+    <child link="link3"/>
+    <origin xyz="0 0 ${link2_len}" rpy="0 0 0"/> <axis xyz="0 1 0"/>
+    <limit lower="-2.5" upper="2.5" effort="2.0" velocity="1.0"/>
+  </joint>
+  <link name="link4">
+    <visual>
+      <geometry>
+        <cylinder radius="${link_radius}" length="${link4_len}"/>
+      </geometry>
+      <origin xyz="0 0 ${link4_len/2}" rpy="0 1.5708 0"/>
+      <material name="grey"/>
+    </visual>
+  </link>
+  <joint name="joint4" type="revolute">
+    <parent link="link3"/>
+    <child link="link4"/>
+    <origin xyz="0 0 ${link3_len}" rpy="0 0 0"/>
+    <axis xyz="0 1 0"/>
+    <limit lower="-1.57" upper="1.57" effort="1.0" velocity="1.0"/>
+  </joint>
+  <link name="link5">
+    <visual>
+      <geometry>
+        <cylinder radius="${link_radius*0.8}" length="${gripper_len}"/>
+      </geometry>
+      <origin xyz="${gripper_len/2} 0 0" rpy="0 1.5708 0"/>
+      <material name="orange"/>
+    </visual>
+  </link>
+  <joint name="joint5" type="revolute">
+    <parent link="link4"/>
+    <child link="link5"/>
+    <origin xyz="0 0 ${link4_len}" rpy="0 0 0"/>
+    <axis xyz="1 0 0"/> <limit lower="-3.14" upper="3.14" effort="1.0" velocity="1.0"/>
+  </joint>
+  <link name="gripper_link">
+    <visual>
+      <geometry>
+        <box size="0.05 0.05 0.05"/>
+      </geometry>
+      <origin xyz="0 0 0" rpy="0 0 0"/>
+      <material name="grey"/>
+    </visual>
+  </link>
+  <joint name="gripper_joint" type="fixed">
+    <parent link="link5"/>
+    <child link="gripper_link"/>
+    <origin xyz="${gripper_len} 0 0" rpy="0 0 0"/>
+  </joint>
+</robot>
